Commit message: Update with recent changes

File: install/dobot_rviz/share/dobot_rviz/urdf/nova5_robot.urdf (robot description, URDF)
Before this commit: robot nova5_robot, 21 links, 20 joints
Links:
- removed link cup_offset_link
- added link calibration_link
- added link tool_link
Joints:
- removed joint cup_offset_joint
- added joint calibration_joint: type fixed, parent Link6, child calibration_link, origin xyz=0 -0.023 0.357 rpy=0 -2.10155463 1.5708
- added joint tool_joint: type fixed, parent Link6, child tool_link, origin xyz=0 0 0.1285 rpy=0 0 0
