Commit message: Update with recent changes

File: src/dobot_rviz/urdf/nova5_robot.urdf (robot description, URDF)
Before this commit: robot nova5_robot, 22 links, 21 joints
Joints:
- joint joint1: limit lower=-6.28 upper=6.28 effort=0 velocity=0 -> lower=-6.2 upper=1 effort=0 velocity=0
- joint joint3: limit lower=-2.79 upper=2.79 effort=0 velocity=0 -> lower=0 upper=2.79 effort=0 velocity=0
